Commit message: feat: add custom pusher end-effector to real robot description
Adds a primitive box+sphere xacro macro plus a fr3_pusher_tcp frame,
mirroring the pusher already modeled in the MuJoCo sim, so the real
robot's URDF carries matching geometry/mass and a TCP frame to plan
and servo against. Selected via ee_id:=custom_pusher_ee hand:=false;
purely additive, default ee_id behavior is unchanged.

File: franka_bringup/urdf/franka_arm.urdf.xacro (robot description, xacro)
@@ -12,4 +12,15 @@
   <!-- ros2_control hardware interface macro -->
   <xacro:include filename="$(find franka_hardware)/ros2_control/franka_arm.ros2_control.xacro"/>
+  <!-- Custom pusher end effector (selected via ee_id:=custom_pusher_ee hand:=false) -->
+  <xacro:include filename="$(find franka_vision_and_manipulation_kit)/accessories/custom_pusher_ee.xacro"/>
+  <xacro:property name="_ee_id_val" value="$(arg ee_id)"/>
+  <xacro:if value="${_ee_id_val == 'custom_pusher_ee'}">
+    <xacro:custom_pusher_ee
+        prefix="${modified_prefix}$(arg robot_type)_"
+        parent="${modified_prefix}$(arg robot_type)_link8"
+        inertials="${xacro.load_yaml('$(find franka_vision_and_manipulation_kit)/accessories/custom_pusher_ee_inertials.yaml')}">
+      <origin xyz="0 0 0" rpy="0 0 0"/>
+    </xacro:custom_pusher_ee>
+  </xacro:if>
   <!-- ros2_control-specific arguments (not declared by description) -->
   <xacro:arg name="robot_ip" default=""/>
