Commit message: feat: add custom plate end-effector to real robot description
Mirrors the existing custom pusher pattern (mount + tilted body + TCP
frame, wired via ee_id:=custom_plate_ee) for a balancing-plate MuJoCo
sim model, so it can be selected on the real FR3 the same way.

Co-Authored-By: Claude Sonnet 5 <noreply@anthropic.com>

File: franka_bringup/urdf/franka_arm.urdf.xacro (robot description, xacro)
@@ -23,4 +23,14 @@
     </xacro:custom_pusher_ee>
   </xacro:if>
+  <!-- Custom plate end effector (selected via ee_id:=custom_plate_ee hand:=false) -->
+  <xacro:include filename="$(find franka_vision_and_manipulation_kit)/accessories/custom_plate_ee.xacro"/>
+  <xacro:if value="${_ee_id_val == 'custom_plate_ee'}">
+    <xacro:custom_plate_ee
+        prefix="${modified_prefix}$(arg robot_type)_"
+        parent="${modified_prefix}$(arg robot_type)_link8"
+        inertials="${xacro.load_yaml('$(find franka_vision_and_manipulation_kit)/accessories/custom_plate_ee_inertials.yaml')}">
+      <origin xyz="0 0 0" rpy="0 0 0"/>
+    </xacro:custom_plate_ee>
+  </xacro:if>
   <!-- ros2_control-specific arguments (not declared by description) -->
   <xacro:arg name="robot_ip" default=""/>

File: franka_fr3_moveit_config/config/fr3_with_pusher.srdf.xacro (robot description, xacro)
@@ -39,3 +39,24 @@
     <disable_collisions link1="fr3_pusher_tip_visual_link" link2="fr3_link8" reason="Adjacent"/>
   </xacro:if>
+  <xacro:if value="${_ee_id_val == 'custom_plate_ee'}">
+    <disable_collisions link1="fr3_plate_mount_link" link2="fr3_plate_link" reason="Adjacent"/>
+    <disable_collisions link1="fr3_plate_mount_link" link2="fr3_link0" reason="Never"/>
+    <disable_collisions link1="fr3_plate_mount_link" link2="fr3_link1" reason="Never"/>
+    <disable_collisions link1="fr3_plate_mount_link" link2="fr3_link2" reason="Never"/>
+    <disable_collisions link1="fr3_plate_mount_link" link2="fr3_link3" reason="Never"/>
+    <disable_collisions link1="fr3_plate_mount_link" link2="fr3_link4" reason="Never"/>
+    <disable_collisions link1="fr3_plate_mount_link" link2="fr3_link5" reason="Never"/>
+    <disable_collisions link1="fr3_plate_mount_link" link2="fr3_link6" reason="Never"/>
+    <disable_collisions link1="fr3_plate_mount_link" link2="fr3_link7" reason="Adjacent"/>
+    <disable_collisions link1="fr3_plate_mount_link" link2="fr3_link8" reason="Adjacent"/>
+    <disable_collisions link1="fr3_plate_link" link2="fr3_link0" reason="Never"/>
+    <disable_collisions link1="fr3_plate_link" link2="fr3_link1" reason="Never"/>
+    <disable_collisions link1="fr3_plate_link" link2="fr3_link2" reason="Never"/>
+    <disable_collisions link1="fr3_plate_link" link2="fr3_link3" reason="Never"/>
+    <disable_collisions link1="fr3_plate_link" link2="fr3_link4" reason="Never"/>
+    <disable_collisions link1="fr3_plate_link" link2="fr3_link5" reason="Never"/>
+    <disable_collisions link1="fr3_plate_link" link2="fr3_link6" reason="Never"/>
+    <disable_collisions link1="fr3_plate_link" link2="fr3_link7" reason="Adjacent"/>
+    <disable_collisions link1="fr3_plate_link" link2="fr3_link8" reason="Adjacent"/>
+  </xacro:if>
 </robot>
